File: ps_adjustable_hv.sch (EAGLE design)
At the start: 40 parts, among them J6 455-1750-1-ND, J7 455-1750-1-ND, X1 DG3XX-02-5.0, X2 DG3XX-02-5.0

Commit message: Start work on new version of adapter
Parts:
- removed J10: (no value), SparkFun-Connectors:CONN_05X2SHD
- added C10: (no value), rcl:C-EUC0805
- added IC1: TL494CN, linear:TL494CN
- added R5: (no value), rcl:R-EU_R0805
Connections:
- removed net 1: C9.-, J10.1, R6.2
- removed net 10: C3.1, J10.10, R4.1
- removed net 3: C4.2, C6.1, J10.3, R1.1, R17.1
- removed net 5: C4.1, J10.5, R2.2, R3.1
- removed net N$16: C3.2, R3.2
- new net COMP: IC1.COMP
- new net N$1: C9.-, IC1.DTC, R6.2
- new net N$12: IC1.RT, R5.1
- new net N$14: C10.2, IC1.CT
- new net N$19: C3.1, IC1.-I1, R4.1
- new net N$20: C4.2, C6.1, IC1.-I2, R1.2, R17.1
- new net N$22: C6.2, R3.2
- new net N$25: C3.2, R2.1
- new net VREF: C9.+, IC1.OUTC, IC1.VREF
- net 2: no longer C9.+, J10.2
- net 7: no longer J10.7
- net 9: now also IC1.+I1; no longer J10.9
- net GND: now also C10.1, IC1.+I2, IC1.E1, IC1.E2, IC1.GND, R5.2; no longer J10.4, J10.6, J10.8
- net N$18: now also C4.1, R2.2, R3.1; no longer C6.2, R2.1
- net N$5: now also R1.1; no longer R1.2
Other:
- moved on the sheet: C3, C4, C5, C6, C9, J6, J7, R1, R17, R2, R3, R4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
